File: LilMix.sch (KiCad schematic (older format))
At the start: 59 parts, among them J1 Conn_01x03, J1_L1 MONO, J1_R1 MONO, J2_L1 MONO, J2_R1 MONO, J3 STEREO, J4 MONO, J5 MONO, J6 STEREO, J7 MONO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

Commit message: Fixed fp on mono jacks.
Parts:
- J1_L1, J1_R1, J2_L1, J2_R1, J7: footprint 4ms-footprints:PJ301M-12 -> Eurocad:PJ301M-12-CC-TIGHT
Changed lines of the file:
@@
 EESchema Schematic File Version 4
-LIBS:LilMix-cache
 EELAYER 30 0
 EELAYER END
@@
 F 0 "J2_R1" H -6128 5934 50  0000 R CNN
 F 1 "MONO" H -6128 6025 50  0000 R CNN
-F 2 "4ms-footprints:PJ301M-12" H -5650 5950 50  0001 C CNN
+F 2 "Eurocad:PJ301M-12-CC-TIGHT" H -5650 5950 50  0001 C CNN
 F 3 "" H -5650 5950 50  0000 C CNN
 	1    -5650 5950
@@
 F 0 "J1_R1" H -6778 5034 50  0000 R CNN
 F 1 "MONO" H -6778 5125 50  0000 R CNN
-F 2 "4ms-footprints:PJ301M-12" H -6300 5050 50  0001 C CNN
+F 2 "Eurocad:PJ301M-12-CC-TIGHT" H -6300 5050 50  0001 C CNN
 F 3 "" H -6300 5050 50  0000 C CNN
 	1    -6300 5050
@@
 F 0 "J1_L1" H -7978 3434 50  0000 R CNN
 F 1 "MONO" H -7978 3525 50  0000 R CNN
-F 2 "4ms-footprints:PJ301M-12" H -7500 3450 50  0001 C CNN
+F 2 "Eurocad:PJ301M-12-CC-TIGHT" H -7500 3450 50  0001 C CNN
 F 3 "" H -7500 3450 50  0000 C CNN
 	1    -7500 3450
@@
 F 0 "J2_L1" H -7328 4234 50  0000 R CNN
 F 1 "MONO" H -7328 4325 50  0000 R CNN
-F 2 "4ms-footprints:PJ301M-12" H -6850 4250 50  0001 C CNN
+F 2 "Eurocad:PJ301M-12-CC-TIGHT" H -6850 4250 50  0001 C CNN
 F 3 "" H -6850 4250 50  0000 C CNN
 	1    -6850 4250
@@
 F 0 "J7" H -7478 1834 50  0000 R CNN
 F 1 "MONO" H -7478 1925 50  0000 R CNN
-F 2 "4ms-footprints:PJ301M-12" H -7000 1850 50  0001 C CNN
+F 2 "Eurocad:PJ301M-12-CC-TIGHT" H -7000 1850 50  0001 C CNN
 F 3 "" H -7000 1850 50  0000 C CNN
 	1    -7000 1850
